File: ECAD/Controller.brd (EAGLE design)
At the start: 100 x 80 mm, 27 parts, among them IC1 PIC18F24K504-I/SP, IC2 TMC2208PLATINE, IC3 ENC28J60PLATINEPCB

Commit message: Reconfigure MCC, try to reduce memory load
Connections:
- removed net N$11: IC1.16
- new net N$1: IC2.4, R5.1
- net MRX: now also R5.2; no longer R5.1
- net MTX: now also IC2.5; no longer R5.2
Changed lines of the file:
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@@
 <signal name="MRX">
 <contactref element="IC1" pad="18"/>
-<contactref element="R5" pad="1"/>
-<wire x1="29.21" y1="40.64" x2="44.87" y2="32.258" width="0" layer="19" extent="1-1"/>
+<contactref element="R5" pad="2"/>
+<wire x1="29.21" y1="40.64" x2="46.57" y2="32.258" width="0" layer="19" extent="1-1"/>
 </signal>
 <signal name="MTX">
 <contactref element="IC1" pad="17"/>
-<contactref element="R5" pad="2"/>
-<wire x1="26.67" y1="40.64" x2="46.57" y2="32.258" width="0" layer="19" extent="1-1"/>
+<contactref element="IC2" pad="5"/>
+<wire x1="19.05" y1="20.32" x2="26.67" y2="40.64" width="0" layer="19" extent="1-1"/>
 </signal>
 <signal name="N$5">
@@
 <wire x1="8.255" y1="12.7" x2="31.75" y2="22.86" width="0" layer="19" extent="1-1"/>
 </signal>
-<signal name="N$11">
-<contactref element="IC1" pad="16"/>
-</signal>
 <signal name="N$13">
 <contactref element="IC1" pad="14"/>
@@
 <contactref element="XPRG" pad="6"/>
 </signal>
+<signal name="N$1">
+<contactref element="R5" pad="1"/>
+<contactref element="IC2" pad="4"/>
+<wire x1="19.05" y1="22.86" x2="44.87" y2="32.258" width="0" layer="19" extent="1-1"/>
+</signal>
 </signals>
